Commit message: something is moving

File: urdf/robot/urdf/materials.xacro (robot description, xacro)
@@ -1,4 +1,4 @@
 <?xml version="1.0" ?>
-<robot name="(Unsaved)" xmlns:xacro="http://www.ros.org/wiki/xacro" >
+<robot name="robot" xmlns:xacro="http://www.ros.org/wiki/xacro" >
 <material name="silver">
   <color rgba="0.700 0.700 0.700 1.000"/>

File: urdf/robot/urdf/robot.xacro (robot description, xacro)
@@ -1,7 +1,7 @@
 <?xml version="1.0" ?>
-<robot name="(Unsaved)" xmlns:xacro="http://www.ros.org/wiki/xacro">
-<xacro:include filename="$(find (Unsaved)_description)/urdf/materials.xacro" />
-<xacro:include filename="$(find (Unsaved)_description)/urdf/(Unsaved).trans" />
-<xacro:include filename="$(find (Unsaved)_description)/urdf/(Unsaved).gazebo" />
+<robot name="robot" xmlns:xacro="http://www.ros.org/wiki/xacro">
+<xacro:include filename="$(find robot)/urdf/materials.xacro" />
+<xacro:include filename="$(find robot)/urdf/robot.trans" />
+<xacro:include filename="$(find robot)/urdf/robot.gazebo" />
 <link name="base_link">
   <inertial>
@@ -13,5 +13,5 @@
     <origin xyz="0 0 0" rpy="0 0 0"/>
     <geometry>
-      <mesh filename="package://(Unsaved)_description/meshes/base_link.stl" scale="0.001 0.001 0.001"/>
+      <mesh filename="package://robot/meshes/base_link.stl" scale="0.001 0.001 0.001"/>
     </geometry>
     <material name="silver"/>
@@ -20,5 +20,5 @@
     <origin xyz="0 0 0" rpy="0 0 0"/>
     <geometry>
-      <mesh filename="package://(Unsaved)_description/meshes/base_link.stl" scale="0.001 0.001 0.001"/>
+      <mesh filename="package://robot/meshes/base_link.stl" scale="0.001 0.001 0.001"/>
     </geometry>
   </collision>
@@ -33,5 +33,5 @@
     <origin xyz="0.08 -0.09 -0.02" rpy="0 0 0"/>
     <geometry>
-      <mesh filename="package://(Unsaved)_description/meshes/right_wheel_1.stl" scale="0.001 0.001 0.001"/>
+      <mesh filename="package://robot/meshes/right_wheel_1.stl" scale="0.001 0.001 0.001"/>
     </geometry>
     <material name="silver"/>
@@ -40,5 +40,5 @@
     <origin xyz="0.08 -0.09 -0.02" rpy="0 0 0"/>
     <geometry>
-      <mesh filename="package://(Unsaved)_description/meshes/right_wheel_1.stl" scale="0.001 0.001 0.001"/>
+      <mesh filename="package://robot/meshes/right_wheel_1.stl" scale="0.001 0.001 0.001"/>
     </geometry>
   </collision>
@@ -53,5 +53,5 @@
     <origin xyz="-0.08 -0.09 -0.02" rpy="0 0 0"/>
     <geometry>
-      <mesh filename="package://(Unsaved)_description/meshes/left_wheel_1.stl" scale="0.001 0.001 0.001"/>
+      <mesh filename="package://robot/meshes/left_wheel_1.stl" scale="0.001 0.001 0.001"/>
     </geometry>
     <material name="silver"/>
@@ -60,5 +60,5 @@
     <origin xyz="-0.08 -0.09 -0.02" rpy="0 0 0"/>
     <geometry>
-      <mesh filename="package://(Unsaved)_description/meshes/left_wheel_1.stl" scale="0.001 0.001 0.001"/>
+      <mesh filename="package://robot/meshes/left_wheel_1.stl" scale="0.001 0.001 0.001"/>
     </geometry>
   </collision>
@@ -73,5 +73,5 @@
     <origin xyz="-0.0 0.06 -0.045" rpy="0 0 0"/>
     <geometry>
-      <mesh filename="package://(Unsaved)_description/meshes/lidar_1.stl" scale="0.001 0.001 0.001"/>
+      <mesh filename="package://robot/meshes/lidar_1.stl" scale="0.001 0.001 0.001"/>
     </geometry>
     <material name="silver"/>
@@ -80,5 +80,5 @@
     <origin xyz="-0.0 0.06 -0.045" rpy="0 0 0"/>
     <geometry>
-      <mesh filename="package://(Unsaved)_description/meshes/lidar_1.stl" scale="0.001 0.001 0.001"/>
+      <mesh filename="package://robot/meshes/lidar_1.stl" scale="0.001 0.001 0.001"/>
     </geometry>
   </collision>
