Commit message: new robot.urdf

File: urdf/robot/urdf/robot.urdf (robot description, URDF)
Before this commit: robot robot, 4 links, 3 joints
Links:
- link base_link: geometry collision mesh filename=file:///Users/karel/Documents/robot/urdf/robot/meshes/base_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 scale=0.001 0.001 0.001; visual mesh filename=file:///Users/karel/Documents/robot/urdf/robot/meshes/base_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 scale=0.001 0.001 0.001
- link left_wheel_1: geometry collision mesh filename=file:///Users/karel/Documents/robot/urdf/robot/meshes/left_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 scale=0.001 0.001 0.001; visual mesh filename=file:///Users/karel/Documents/robot/urdf/robot/meshes/left_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 scale=0.001 0.001 0.001
- link lidar_1: geometry collision mesh filename=file:///Users/karel/Documents/robot/urdf/robot/meshes/lidar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 scale=0.001 0.001 0.001; visual mesh filename=file:///Users/karel/Documents/robot/urdf/robot/meshes/lidar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 scale=0.001 0.001 0.001
- link right_wheel_1: geometry collision mesh filename=file:///Users/karel/Documents/robot/urdf/robot/meshes/right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 scale=0.001 0.001 0.001; visual mesh filename=file:///Users/karel/Documents/robot/urdf/robot/meshes/right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 scale=0.001 0.001 0.001

Commit message: kind of working

File: urdf/robot/urdf/robot.urdf (robot description, URDF)
Before this commit: robot robot, 4 links, 3 joints
Links:
- link base_link: geometry collision mesh filename=file:///home/john/robot/urdf/robot/meshes/base_link.stl scale=0.001 0.001 0.001; visual mesh filename=file:///home/john/robot/urdf/robot/meshes/base_link.stl scale=0.001 0.001 0.001
- link left_wheel_1: geometry collision mesh filename=file:///home/john/robot/urdf/robot/meshes/left_wheel_1.stl scale=0.001 0.001 0.001; visual mesh filename=file:///home/john/robot/urdf/robot/meshes/left_wheel_1.stl scale=0.001 0.001 0.001
- link lidar_1: geometry collision mesh filename=file:///home/john/robot/urdf/robot/meshes/lidar_1.stl scale=0.001 0.001 0.001; visual mesh filename=file:///home/john/robot/urdf/robot/meshes/lidar_1.stl scale=0.001 0.001 0.001
- link right_wheel_1: geometry collision mesh filename=file:///home/john/robot/urdf/robot/meshes/right_wheel_1.stl scale=0.001 0.001 0.001; visual mesh filename=file:///home/john/robot/urdf/robot/meshes/right_wheel_1.stl scale=0.001 0.001 0.001

Commit message: urdf fix

File: urdf/robot/urdf/robot.urdf (robot description, URDF)
Before this commit: robot robot, 4 links, 3 joints
Links:
- link left_wheel_1: geometry collision mesh filename=file:///Users/karel/Documents/robot/urdf/robot/meshes/left_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 scale=0.0001 0.0001 0.0001; visual mesh filename=file:///Users/karel/Documents/robot/urdf/robot/meshes/left_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 scale=0.0001 0.0001 0.0001
- link lidar_1: geometry collision mesh filename=file:///Users/karel/Documents/robot/urdf/robot/meshes/lidar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 scale=0.0001 0.0001 0.0001; visual mesh filename=file:///Users/karel/Documents/robot/urdf/robot/meshes/lidar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 scale=0.0001 0.0001 0.0001
- link right_wheel_1: geometry collision mesh filename=file:///Users/karel/Documents/robot/urdf/robot/meshes/right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 scale=0.0001 0.0001 0.0001; visual mesh filename=file:///Users/karel/Documents/robot/urdf/robot/meshes/right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 scale=0.0001 0.0001 0.0001

Commit message: caster wheel urdf

File: urdf/robot/urdf/robot.urdf (robot description, URDF)
Before this commit: robot robot, 4 links, 3 joints
Links:
- removed link lidar_1
- added link caster_fork_1, mass 0.001842425119376973; collision mesh filename=file:///Users/karel/Documents/robot/urdf/robot/meshes/caste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 scale=0.001 0.001 0.001; visual mesh filename=file:///Users/karel/Documents/robot/urdf/robot/meshes/caste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 scale=0.001 0.001 0.001
- added link caster_wheel_1, mass 0.0016434456569091604; collision mesh filename=file:///Users/karel/Documents/robot/urdf/robot/meshes/caste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 scale=0.001 0.001 0.001; visual mesh filename=file:///Users/karel/Documents/robot/urdf/robot/meshes/caste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 scale=0.001 0.001 0.001
- link base_link: mass 1.2850428455001501 -> 1.2728533351045312
- link left_wheel_1: geometry collision mesh filename=file:///Users/karel/Documents/robot/urdf/robot/meshes/left_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 scale=0.001 0.001 0.001; visual mesh filename=file:///Users/karel/Documents/robot/urdf/robot/meshes/left_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 scale=0.001 0.001 0.001
- link right_wheel_1: geometry collision mesh filename=file:///Users/karel/Documents/robot/urdf/robot/meshes/right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 scale=0.001 0.001 0.001; visual mesh filename=file:///Users/karel/Documents/robot/urdf/robot/meshes/right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 scale=0.001 0.001 0.001
Joints:
- added joint Revolute 4: type continuous, parent base_link, child right_wheel_1, origin xyz=-0.08 0.08 0.02 rpy=0 0 0, axis -1.0 0.0 0.0
- joint Revolute 1: child right_wheel_1 -> caster_wheel_1; origin xyz=-0.08 0.09 0.02 rpy=0 0 0 -> xyz=0.005 0.008443 -0.0115 rpy=0 0 0; parent base_link -> caster_fork_1
- joint Revolute 2: axis 1.0 0.0 0.0 -> 0.0 0.0 -1.0; child left_wheel_1 -> caster_fork_1; origin xyz=0.08 0.09 0.02 rpy=0 0 0 -> xyz=0.0 -0.08 -0.001 rpy=0 0 0
- joint Revolute 3: axis 0.0 0.0 1.0 -> 1.0 0.0 0.0; child lidar_1 -> left_wheel_1; origin xyz=0.0 -0.06 0.045 rpy=0 0 0 -> xyz=0.08 0.08 0.02 rpy=0 0 0

File: urdf/robot/urdf/robot.xacro (robot description, xacro)
@@ -6,7 +6,7 @@
 <link name="base_link">
   <inertial>
-    <origin xyz="1.355046717905403e-13 0.009343506444008564 0.019993521445171167" rpy="0 0 0"/>
-    <mass value="1.2850428455001501"/>
-    <inertia ixx="0.004491" iyy="0.002568" izz="0.006705" ixy="0.0" iyz="-2e-06" ixz="0.0"/>
+    <origin xyz="-1.514808277263353e-17 5.101665553979481e-05 0.019999664794410715" rpy="0 0 0"/>
+    <mass value="1.2728533351045312"/>
+    <inertia ixx="0.004415" iyy="0.00256" izz="0.006635" ixy="0.0" iyz="-0.0" ixz="0.0"/>
   </inertial>
   <visual>
@@ -24,21 +24,41 @@
   </collision>
 </link>
-<link name="right_wheel_1">
+<link name="caster_wheel_1">
   <inertial>
-    <origin xyz="-0.009999999999999995 0.0 0.0" rpy="0 0 0"/>
-    <mass value="0.09349379737083224"/>
-    <inertia ixx="7.5e-05" iyy="4.1e-05" izz="4.1e-05" ixy="-0.0" iyz="0.0" ixz="0.0"/>
+    <origin xyz="-0.005000000000000495 -2.058718588243691e-07 -2.149933009398808e-12" rpy="0 0 0"/>
+    <mass value="0.0016434456569091604"/>
+    <inertia ixx="0.0" iyy="0.0" izz="0.0" ixy="0.0" iyz="0.0" ixz="0.0"/>
   </inertial>
   <visual>
-    <origin xyz="0.08 -0.09 -0.02" rpy="0 0 0"/>
+    <origin xyz="-0.005 0.071557 0.0125" rpy="0 0 0"/>
     <geometry>
-      <mesh filename="package://robot/meshes/right_wheel_1.stl" scale="0.001 0.001 0.001"/>
+      <mesh filename="package://robot/meshes/caster_wheel_1.stl" scale="0.001 0.001 0.001"/>
     </geometry>
     <material name="silver"/>
   </visual>
   <collision>
-    <origin xyz="0.08 -0.09 -0.02" rpy="0 0 0"/>
+    <origin xyz="-0.005 0.071557 0.0125" rpy="0 0 0"/>
     <geometry>
-      <mesh filename="package://robot/meshes/right_wheel_1.stl" scale="0.001 0.001 0.001"/>
+      <mesh filename="package://robot/meshes/caster_wheel_1.stl" scale="0.001 0.001 0.001"/>
+    </geometry>
+  </collision>
+</link>
+<link name="caster_fork_1">
+  <inertial>
+    <origin xyz="-4.828898138961918e-16 0.003917233985619384 -0.006001009388864729" rpy="0 0 0"/>
+    <mass value="0.001842425119376973"/>
+    <inertia ixx="0.0" iyy="0.0" izz="0.0" ixy="-0.0" iyz="0.0" ixz="-0.0"/>
+  </inertial>
+  <visual>
+    <origin xyz="-0.0 0.08 0.001" rpy="0 0 0"/>
+    <geometry>
+      <mesh filename="package://robot/meshes/caster_fork_1.stl" scale="0.001 0.001 0.001"/>
+    </geometry>
+    <material name="silver"/>
+  </visual>
+  <collision>
+    <origin xyz="-0.0 0.08 0.001" rpy="0 0 0"/>
+    <geometry>
+      <mesh filename="package://robot/meshes/caster_fork_1.stl" scale="0.001 0.001 0.001"/>
     </geometry>
   </collision>
@@ -51,5 +71,5 @@
   </inertial>
   <visual>
-    <origin xyz="-0.08 -0.09 -0.02" rpy="0 0 0"/>
+    <origin xyz="-0.08 -0.08 -0.02" rpy="0 0 0"/>
     <geometry>
       <mesh filename="package://robot/meshes/left_wheel_1.stl" scale="0.001 0.001 0.001"/>
@@ -58,5 +78,5 @@
   </visual>
   <collision>
-    <origin xyz="-0.08 -0.09 -0.02" rpy="0 0 0"/>
+    <origin xyz="-0.08 -0.08 -0.02" rpy="0 0 0"/>
     <geometry>
       <mesh filename="package://robot/meshes/left_wheel_1.stl" scale="0.001 0.001 0.001"/>
@@ -64,41 +84,47 @@
   </collision>
 </link>
-<link name="lidar_1">
+<link name="right_wheel_1">
   <inertial>
-    <origin xyz="-3.769546289141946e-18 0.0 0.015" rpy="0 0 0"/>
-    <mass value="0.039961058553662165"/>
-    <inertia ixx="7e-06" iyy="7e-06" izz="8e-06" ixy="0.0" iyz="0.0" ixz="-0.0"/>
+    <origin xyz="-0.009999999999999995 0.0 0.0" rpy="0 0 0"/>
+    <mass value="0.09349379737083224"/>
+    <inertia ixx="7.5e-05" iyy="4.1e-05" izz="4.1e-05" ixy="-0.0" iyz="0.0" ixz="0.0"/>
   </inertial>
   <visual>
-    <origin xyz="-0.0 0.06 -0.045" rpy="0 0 0"/>
+    <origin xyz="0.08 -0.08 -0.02" rpy="0 0 0"/>
     <geometry>
-      <mesh filename="package://robot/meshes/lidar_1.stl" scale="0.001 0.001 0.001"/>
+      <mesh filename="package://robot/meshes/right_wheel_1.stl" scale="0.001 0.001 0.001"/>
     </geometry>
     <material name="silver"/>
   </visual>
   <collision>
-    <origin xyz="-0.0 0.06 -0.045" rpy="0 0 0"/>
+    <origin xyz="0.08 -0.08 -0.02" rpy="0 0 0"/>
     <geometry>
-      <mesh filename="package://robot/meshes/lidar_1.stl" scale="0.001 0.001 0.001"/>
+      <mesh filename="package://robot/meshes/right_wheel_1.stl" scale="0.001 0.001 0.001"/>
     </geometry>
   </collision>
 </link>
 <joint name="Revolute 1" type="continuous">
-  <origin xyz="-0.08 0.09 0.02" rpy="0 0 0"/>
+  <origin xyz="0.005 0.008443 -0.0115" rpy="0 0 0"/>
+  <parent link="caster_fork_1"/>
+  <child link="caster_wheel_1"/>
+  <axis xyz="-1.0 0.0 0.0"/>
+</joint>
+<joint name="Revolute 2" type="continuous">
+  <origin xyz="0.0 -0.08 -0.001" rpy="0 0 0"/>
+  <parent link="base_link"/>
+  <child link="caster_fork_1"/>
+  <axis xyz="0.0 0.0 -1.0"/>
+</joint>
+<joint name="Revolute 3" type="continuous">
+  <origin xyz="0.08 0.08 0.02" rpy="0 0 0"/>
+  <parent link="base_link"/>
+  <child link="left_wheel_1"/>
+  <axis xyz="1.0 0.0 0.0"/>
+</joint>
+<joint name="Revolute 4" type="continuous">
+  <origin xyz="-0.08 0.08 0.02" rpy="0 0 0"/>
   <parent link="base_link"/>
   <child link="right_wheel_1"/>
   <axis xyz="-1.0 0.0 0.0"/>
 </joint>
-<joint name="Revolute 2" type="continuous">
-  <origin xyz="0.08 0.09 0.02" rpy="0 0 0"/>
-  <parent link="base_link"/>
-  <child link="left_wheel_1"/>
-  <axis xyz="1.0 0.0 0.0"/>
-</joint>
-<joint name="Revolute 3" type="continuous">
-  <origin xyz="0.0 -0.06 0.045" rpy="0 0 0"/>
-  <parent link="base_link"/>
-  <child link="lidar_1"/>
-  <axis xyz="0.0 0.0 1.0"/>
-</joint>
 </robot>

Commit message: working

File: urdf/robot/urdf/robot.urdf (robot description, URDF)
Before this commit: robot robot, 5 links, 4 joints
Links:
- link base_link: geometry collision mesh filename=file:///home/john/robot/urdf/robot/meshes/base_link.stl scale=0.001 0.001 0.001; visual mesh filename=file:///home/john/robot/urdf/robot/meshes/base_link.stl scale=0.001 0.001 0.001
- link caster_fork_1: geometry collision mesh filename=file:///home/john/robot/urdf/robot/meshes/caster_fork_1.stl scale=0.001 0.001 0.001; visual mesh filename=file:///home/john/robot/urdf/robot/meshes/caster_fork_1.stl scale=0.001 0.001 0.001
- link caster_wheel_1: geometry collision mesh filename=file:///home/john/robot/urdf/robot/meshes/caster_wheel_1.stl scale=0.001 0.001 0.001; visual mesh filename=file:///home/john/robot/urdf/robot/meshes/caster_wheel_1.stl scale=0.001 0.001 0.001
- link left_wheel_1: geometry collision mesh filename=file:///home/john/robot/urdf/robot/meshes/left_wheel_1.stl scale=0.001 0.001 0.001; visual mesh filename=file:///home/john/robot/urdf/robot/meshes/left_wheel_1.stl scale=0.001 0.001 0.001
- link right_wheel_1: geometry collision mesh filename=file:///home/john/robot/urdf/robot/meshes/right_wheel_1.stl scale=0.001 0.001 0.001; visual mesh filename=file:///home/john/robot/urdf/robot/meshes/right_wheel_1.stl scale=0.001 0.001 0.001

Commit message: added camera

File: urdf/robot/urdf/robot.urdf (robot description, URDF)
Before this commit: robot robot, 5 links, 4 joints
Links:
- added link camera_link, mass 0.01; collision box size=0.02 0.02 0.02; visual box size=0.02 0.02 0.02
- link base_link: geometry collision mesh filename=meshes/base_link.stl scale=0.001 0.001 0.001; visual mesh filename=meshes/base_link.stl scale=0.001 0.001 0.001
- link caster_fork_1: geometry collision mesh filename=meshes/caster_fork_1.stl scale=0.001 0.001 0.001; visual mesh filename=meshes/caster_fork_1.stl scale=0.001 0.001 0.001
- link caster_wheel_1: geometry collision mesh filename=meshes/caster_wheel_1.stl scale=0.001 0.001 0.001; visual mesh filename=meshes/caster_wheel_1.stl scale=0.001 0.001 0.001
- link left_wheel_1: geometry collision mesh filename=meshes/left_wheel_1.stl scale=0.001 0.001 0.001; visual mesh filename=meshes/left_wheel_1.stl scale=0.001 0.001 0.001
- link right_wheel_1: geometry collision mesh filename=meshes/right_wheel_1.stl scale=0.001 0.001 0.001; visual mesh filename=meshes/right_wheel_1.stl scale=0.001 0.001 0.001
Joints:
- added joint camera_joint: type fixed, parent base_link, child camera_link, origin xyz=0 -0.09 0.05 rpy=0 0 0
