Commit message: urdf mass change and training cleaner

File: sim/balance/balance.urdf (robot description, URDF)
Before this commit: robot balance, 4 links, 3 joints
Links:
- link balance_wheel_1: mass 0.9154342382147101 -> 2.5
- link base_link: mass 1.1691157163837433 -> 3
- link left_wheel_1: mass 0.9154342382147101 -> 2.5
- link right_wheel_1: mass 0.9154342382147101 -> 2.5
